File: MCU Datalogger.kicad_sch (KiCad schematic)
At the start: 0 parts

Commit message: Complete initial schematic design -2 layer
Parts:
- added BT1: Battery, Connector_PinHeader_2.54mm:PinHeader_1x02_P2.54mm_Vertical, symbol Device:Battery
- added C1, C2: 22pF, Capacitor_SMD:C_0805_2012Metric, symbol Device:C
- added C3: 100nF, Capacitor_SMD:C_0805_2012Metric, symbol Device:C_Polarized
- added C4, C5: 0.1uF, Capacitor_SMD:C_0805_2012Metric, symbol Device:C
- added D1, D2: LED, LED_SMD:LED_0805_2012Metric, symbol Device:LED
- added H1, H2, H3, H4: MountingHole, MountingHole:MountingHole_2.1mm, symbol Mechanical:MountingHole
- added R1, R4: 330, Resistor_SMD:R_0805_2012Metric, symbol Device:R
- added R2, R3: 4.7k, Resistor_SMD:R_0805_2012Metric, symbol Device:R
- added R5, R6, R7: 10k, Resistor_SMD:R_0805_2012Metric, symbol Device:R
- added U1, U3: 24LC1025, Package_SO:SOIC-8_5.3x5.3mm_P1.27mm, symbol Memory_EEPROM:24LC1025
- added U2: DS1337S_, DS1337S_:SOIC127P600X175-8N, symbol DS1337S_:DS1337S_
- added U4: ATMEGA328P-AU, ATMEGA328P-AU(1):QFP80P900X900X120-32N, symbol ATMEGA328P-AU(2):ATMEGA328P-AU
- added Y1: 32.768MHz, Crystal:Crystal_SMD_5032-2Pin_5.0x3.2mm_HandSoldering, symbol Device:Crystal
- added Y2: 16MHz, Crystal:Crystal_SMD_5032-2Pin_5.0x3.2mm_HandSoldering, symbol Device:Crystal
Connections:
- new net: C1.2, U4.7 (PB6), Y2.2
- new net: C4.2, U4.20 (AREF)
- new net: R6.2, U2.7 (SQW/~INT)
- new net: C2.2, U4.8 (PB7), Y2.1
- new net: D2.1 (K), R1.1
- new net: D1.1 (K), R4.2
- new net: U2.1 (X1), Y1.2
- new net: U2.2 (X2), Y1.1
- new net: R5.2, U2.3 (~{INTA})
- new net D2: U4.32 (PD2)
- new net D3: U4.1 (PD3)
- new net D4: U4.2 (PD4)
- new net D5: U4.9 (PD5)
- new net D6: U4.10 (PD6)
- new net D7: U4.11 (PD7)
- new net DB: U4.12 (PB0)
- new net GND: BT1.2 (-), C1.1, C2.1, C3.2, C4.1, C5.2, R1.2, R4.1, U1.4 (GND), U1.7 (WP), U2.4 (GND), U3.2 (A1), U3.4 (GND), U3.7 (WP), U4.21 (GND), U4.3 (GND), U4.5 (GND)
- new net MISO: U4.16 (PB4)
- new net MOSI: U4.15 (PB3)
- new net RESET: R7.2, U4.29 (PC6/~{RESET})
- new net RX: U4.30 (PD0)
- new net SCK: D1.2 (A), R2.2, U1.6 (SCL), U2.6 (SCL), U3.6 (SCL), U4.17 (PB5), U4.28 (PC5)
- new net SDA: R3.2, U1.5 (SDA), U2.5 (SDA), U3.5 (SDA), U4.27 (PC4)
- new net TX: U4.31 (PD1)
- new net VCC: BT1.1 (+), C3.1, C5.1, D2.2 (A), R2.1, R3.1, R5.1, R6.1, R7.1, U1.1 (A0), U1.2 (A1), U1.3 (A2), U1.8 (VCC), U2.8 (VCC), U3.1 (A0), U3.3 (A2), U3.8 (VCC), U4.18 (AVCC), U4.4 (VCC), U4.6 (VCC)
- no-connect marks 0 -> 9
Other:
- added sheet Connector Sheet (connector.kicad_sch)

Commit message: Added a page setting
Other:
- title: (none) -> MCU-DATALOGGER
Changed lines of the file:
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@@
 	(generator_version "10.0")
 	(paper "A4")
+	(title_block
+		(title "MCU-DATALOGGER")
+		(date "2026-10-21")
+		(rev "1")
+	)
 	(text_box "Clock"
 		(exclude_from_sim no)

Commit message: Set up of EEschema
Other:
- title: MCU-DATALOGGER -> ${project_name}
Changed lines of the file:
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@@
 	(paper "A4")
 	(title_block
-		(title "MCU-DATALOGGER")
+		(title "${project_name}")
 		(date "2026-10-21")
 		(rev "1")
